File: PCB/_Sliders/sliders/sliders.kicad_sch (KiCad schematic)
At the start: 14 parts, among them J1 OLED, J2 OLED, J3 Magnetic connector, J4 Magnetic connector, J5 Magnetic connector, J6 Magnetic connector, SW1 RST, U1 SuperMini_NRF52840

Commit message: PCB V2 design
Parts:
- removed H1, H2, H3, H4: MountingHole, MountingHole:MountingHole_3.2mm_M3, symbol Mechanical:MountingHole
Other:
- removed sheet Switch Matrix
- company: KillrOfLife -> (none)
- title: Macro32 -> (none)
- moved on the sheet: J1, J2, J3, J4, J5, J6, R1, R2, SW1, U1
