File: PCB/macro32/macro32_matrix.kicad_sch (KiCad schematic)
At the start: 44 parts

Commit message: fix schema header
Other:
- company: KillrOfLife -> Lucid-void
Changed lines of the file:
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@@
 	(title_block
 		(title "Macro32")
-		(date "2025-11-08")
+		(date "2026-07-16")
 		(rev "v2")
-		(company "KillrOfLife")
+		(company "Lucid-void")
 	)
 	(junction
