File: PCB/macro32/macro32_neopixels.kicad_sch (KiCad schematic)
At the start: 10 parts, among them U4 74AHC1G125

Commit message: fix schema header
Other:
- company: (none) -> Lucid-void
- title: (none) -> Macro32
Changed lines of the file:
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@@
 	(generator_version "10.0")
 	(paper "A4")
+	(title_block
+		(title "Macro32")
+		(date "2026-07-16")
+		(rev "v2")
+		(company "Lucid-void")
+	)
 	(junction
 		(at 123.19 105.41)
